File: _autosave-smart_wristband.kicad_sch (KiCad schematic)
At the start: 18 parts, among them J1 USB_B_Micro, J2 Conn_01x04_Male, J3 Conn_01x02_Male, J4 Conn_01x02_Male, U1 STM32F042F6Px, U2 DS1307Z+, U3 LSM6DS3, U4 MCP1700-3302E_SOT23, Y1 Crystal

Commit message: add alot
Parts:
- removed J3: Conn_01x02_Male, Connector_PinSocket_2.00mm:PinSocket_1x02_P2.00mm_Vertical, symbol Connector:Conn_01x02_Male
- added C10: C, Capacitor_SMD:C_0402_1005Metric, symbol Device:C
- added C11, C12: C, Capacitor_SMD:C_0603_1608Metric, symbol Device:C
- added C13, C5, C8: C, Capacitor_SMD:C_0603_1608Metric_Pad1.05x0.95mm_HandSolder, symbol Device:C
- added D1, D2: LED, LED_SMD:LED_0603_1608Metric, symbol Device:LED
- added IC1: TP4056, Package_SO:Diodes_PSOP-8, symbol New_Library:TP4056
- added IC2: DW01A, drone_v3:SOT23-6, symbol New_Library:DW01A
- added J3, J5: Conn_01x04_Male, Connector_JST:JST_SH_BM04B-SRSS-TB_1x04-1MP_P1.00mm_Vertical, symbol Connector:Conn_01x04_Male
- added Q1: FS8205A, drone_v3:SOP65P640X120-8N, symbol New_Library:FS8205A
- added R3, R4, R5, R6, R7: R, Resistor_SMD:R_0603_1608Metric, symbol Device:R
- added SW1: SW_DPST_x2, drone_v3:TouchSlider-2_10x10mm, symbol Switch:SW_DPST_x2
- C3, C4: footprint Capacitor_SMD:C_0402_1005Metric -> Capacitor_SMD:C_0603_1608Metric_Pad1.05x0.95mm_HandSolder
Connections:
- net +3V3: now also U1.4 (NRST), C12.1, J3.4 (Pin_4), J5.1 (Pin_1); no longer J4.2 (Pin_2), U4.1 (GND)
- net +5V: now also C5.1, IC1.4 (VCC), IC1.8 (CE), R6.1, R7.1
- net CAP_Touch: now also U1.13 (PA7), SW1.1 (A)
- net GND: now also J4.1 (Pin_1), U4.1 (GND), C10.2, C11.2, C12.2, C13.2, C5.2, C8.2, IC1.1 (TEMP), IC1.3 (GND), IC2.6 (GND), J3.1 (Pin_1), J5.4 (Pin_4), Q1.1, Q1.2, Q1.3, Q1.6, Q1.7, Q1.8, R3.2, R5.2
- net USB_DM: now also J5.2 (Pin_2)
- net USB_DP: now also J5.3 (Pin_3)
- net Vdrive: now reaches U4.3 (VI)
- net Vdrive: now also C11.1, C8.1, R4.1; no longer J4.1 (Pin_1)
- net CAP_sample: now reaches U1.11 (PA5)
- net CAP_sample: now also C13.1
- net CAP_Touch1: now reaches U1.12 (PA6)
- net CAP_Touch1: now also SW1.2 (B)
- net SWCLK: now reaches U1.19 (PA13)
- net SWCLK: now also J3.2 (Pin_2)
- net SWDIO: now reaches U1.20 (PA14)
- net SWDIO: now also J3.3 (Pin_3)
- net TX: now reaches U1.8 (PA2)
- net RX: now reaches U1.9 (PA3)
- new net: IC2.5 (VCC), R4.2
- new net: IC2.1 (OD), Q1.4
- new net: IC2.2 (CS), R5.1
- new net: IC2.3 (OC), Q1.5
- new net: D2.2 (A), R7.2
- new net: D1.1 (K), IC1.7 (CHRG)
- new net: D1.2 (A), R6.2
- new net: C10.1, IC1.5 (BAT), J4.2 (Pin_2)
- new net: IC1.2 (PROG), R3.1
- new net: D2.1 (K), IC1.6 (STDBY)
Other:
- moved on the sheet: C7, C9, J1, J2, J4, U3, U4
