File: smart_wristband.kicad_pcb (KiCad board)
At the start: 2 copper layers, 37.5 x 11.5 mm, 16 parts, among them J1 USB_B_Micro, J2 Conn_01x04_Male, J3 Conn_01x02_Male, J4 Conn_01x02_Male, U1 STM32F042F6Px, U2 DS1307Z+, U3 LSM6DS3, U4 MCP1700-3302E_SOT23, Y1 Crystal

Commit message: add alot
Parts:
- added C10: C, Capacitor_SMD:C_0402_1005Metric, B.Cu at (120.6, 92.5)
- added C11: C, Capacitor_SMD:C_0603_1608Metric, F.Cu at (116.7, 100.3)
- added C12: C, Capacitor_SMD:C_0603_1608Metric, F.Cu at (112.3, 100.8)
- added C13: C, Capacitor_SMD:C_0603_1608Metric_Pad1.05x0.95mm_HandSolder, F.Cu at (133.2, 101.0)
- added C5: C, Capacitor_SMD:C_0603_1608Metric_Pad1.05x0.95mm_HandSolder, B.Cu at (129.2, 97.2)
- added C8: C, Capacitor_SMD:C_0603_1608Metric_Pad1.05x0.95mm_HandSolder, B.Cu at (114.2, 100.3)
- added D1: LED, LED_SMD:LED_0603_1608Metric, B.Cu at (126.2, 92.3)
- added D2: LED, LED_SMD:LED_0603_1608Metric, B.Cu at (123.0, 92.1)
- added G***: LOGO, drone_v3:pusheen, B.Cu at (139.5, 97.5)
- added IC1: TP4056, Package_SO:Diodes_PSOP-8, B.Cu at (124.4, 95.7)
- added IC2: DW01A, drone_v3:SOT23-6, B.Cu at (116.0, 96.0)
- added J5: Conn_01x04_Male, Connector_JST:JST_SH_BM04B-SRSS-TB_1x04-1MP_P1.00mm_Vertical, B.Cu at (138.3, 93.4)
- added Q1: FS8205A, drone_v3:SOP65P640X120-8N, B.Cu at (123.3, 100.3)
- added R3: R, Resistor_SMD:R_0603_1608Metric, B.Cu at (120.0, 97.0)
- added R4: R, Resistor_SMD:R_0603_1608Metric, B.Cu at (112.7, 100.4)
- added R5: R, Resistor_SMD:R_0603_1608Metric, B.Cu at (115.8, 98.4)
- added R6: R, Resistor_SMD:R_0603_1608Metric, B.Cu at (129.9, 92.1)
- added R7: R, Resistor_SMD:R_0603_1608Metric, B.Cu at (133.0, 92.1)
- added SW1: SW_DPST_x2, drone_v3:TouchSlider-2_10x10mm, F.Cu at (141.3, 96.6)
- C3, C4: footprint Capacitor_SMD:C_0402_1005Metric -> Capacitor_SMD:C_0603_1608Metric_Pad1.05x0.95mm_HandSolder
- J3: value Conn_01x02_Male -> Conn_01x04_Male; footprint Connector_PinSocket_2.00mm:PinSocket_1x02_P2.00mm_Vertical -> Connector_JST:JST_SH_BM04B-SRSS-TB_1x04-1MP_P1.00mm_Vertical
- J4: moved to B.Cu
- moved J3 12.5 mm to (121.7, 93.2), turned to 0 degrees
- moved U4 11.6 mm to (114.5, 100.8)
- moved C3 6.29 mm to (106.4, 100.5), turned to 90 degrees
- moved C4 4.70 mm to (111.0, 100.4), turned to 90 degrees
- moved C2 1.34 mm to (116.8, 98.2), turned to 90 degrees
- moved C6 1.16 mm to (126.6, 98.9)
- moved U1 0.93 mm to (121.3, 99.1)
- moved Y1 0.70 mm to (109.6, 100.3)
- moved J4 0.49 mm to (117.0, 92.7), turned to -90 degrees
- moved J2 0.17 mm to (104.1, 92.8)
Connections:
- net Net-(U1-Pad8) renamed TX
- net Net-(U1-Pad9) renamed RX
- J3 pad 1: +5V -> GND
- J3 pad 2: GND -> SWCLK
- J4 pad 1: Net-(J4-Pad1) -> GND
- J4 pad 2: +3V3 -> Net-(C10-Pad1)
- U1 pad 11: Net-(U1-Pad11) -> CAP_sample
- U1 pad 12: Net-(U1-Pad12) -> CAP_Touch1
- U1 pad 13: Net-(U1-Pad13) -> CAP_Touch
- U1 pad 19: Net-(U1-Pad19) -> SWCLK
- U1 pad 20: Net-(U1-Pad20) -> SWDIO
- U1 pad 4: Net-(U1-Pad4) -> +3V3
- U4 pad 1: +3V3 -> GND
- U4 pad 3: Net-(J4-Pad1) -> Vdrive
Routing:
- net +3V3: track 0.00 -> 90.5 mm, vias 0 -> 1
- net GND: track 0.00 -> 71.7 mm, vias 0 -> 18
- net +5V: track 0.00 -> 28.3 mm, vias 0 -> 1
- net CAP_Touch: track 0.00 -> 17.6 mm, vias 0 -> 1
- net USB_DM: track 2.16 -> 19.4 mm, vias 0 -> 1
- net Net-(IC2-Pad1): track 0.00 -> 16.8 mm
- net USB_DP: track 1.24 -> 17.4 mm, vias 0 -> 1
- net CAP_Touch1: track 0.00 -> 15.9 mm, vias 0 -> 1
- net Net-(D2-Pad2): track 0.00 -> 12.8 mm
- net Net-(D2-Pad1): track 0.00 -> 11.6 mm
- net Net-(C10-Pad1): track 0.00 -> 10.9 mm
- net CAP_sample: track 0.00 -> 9.67 mm
- net Net-(IC2-Pad5): track 0.00 -> 9.35 mm
- net Net-(IC2-Pad3): track 0.00 -> 7.76 mm
- net SDA: track 18.4 -> 25.5 mm, vias 0 -> 2
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- added copper zone on B.Cu, net GND
- added copper zone on F.Cu, net GND
Other:
- board size 37.5 x 11.5 mm -> 45 x 11.5 mm
